Commit message: student distillation training complete,  evaluation successful

File: dextrah_lab/assets/kuka_inspirehand/urdf/combined.urdf (robot description, URDF)
Before this commit: robot lbr_iiwa7_r800, 21 links, 20 joints
Links:
- removed link Link13
- removed link Link14
- removed link Link23
- removed link Link24
- removed link Link3
- removed link Link33
- removed link Link34
- removed link Link4
- removed link Link43
- removed link Link44
- removed link Link47
- removed link Link48
- added link index_link_0, mass 0.0042403; collision mesh filename=./meshes/index_link_0.STL; visual mesh filename=./meshes/index_link_0.STL
- added link index_link_1, mass 0.0045683; collision mesh filename=./meshes/index_link_1.STL; visual mesh filename=./meshes/index_link_1.STL
- added link inspirehand_mount, mass 0.05; collision box size=0.001 0.001 0.001; visual box size=0.001 0.001 0.001
- added link little_link_0, mass 0.0042403; collision mesh filename=./meshes/little_link_0.STL; visual mesh filename=./meshes/little_link_0.STL
- added link little_link_1, mass 0.0035996; collision mesh filename=./meshes/little_link_1.STL; visual mesh filename=./meshes/little_link_1.STL
- added link middle_link_0, mass 0.0042403; collision mesh filename=./meshes/middle_link_0.STL; visual mesh filename=./meshes/middle_link_0.STL
- added link middle_link_1, mass 0.0050396; collision mesh filename=./meshes/middle_link_1.STL; visual mesh filename=./meshes/middle_link_1.STL
- added link ring_link_0, mass 0.0042403; collision mesh filename=./meshes/ring_link_0.STL; visual mesh filename=./meshes/ring_link_0.STL
- added link ring_link_1, mass 0.0045683; collision mesh filename=./meshes/ring_link_1.STL; visual mesh filename=./meshes/ring_link_1.STL
- added link thumb_link_0, mass 0.0018869; collision mesh filename=./meshes/thumb_link_0.STL; visual mesh filename=./meshes/thumb_link_0.STL
- added link thumb_link_1, mass 0.0066075; collision mesh filename=./meshes/thumb_link_1.STL; visual mesh filename=./meshes/thumb_link_1.STL
- added link thumb_link_2, mass 0.0037847; collision mesh filename=./meshes/thumb_link_2.STL; visual mesh filename=./meshes/thumb_link_2.STL
- added link thumb_link_3, mass 0.0033441; collision mesh filename=./meshes/thumb_link_3.STL; visual mesh filename=./meshes/thumb_link_3.STL
Joints:
- added joint inspirehand_mount_joint: type fixed, parent inspirehand_mount, child palm, origin xyz=0 0 0 rpy=0 0 0
- joint iiwa7_hand_fixed: child palm -> inspirehand_mount
- joint index_joint_0: child Link3 -> index_link_0
- joint index_joint_1: child Link4 -> index_link_1; parent Link3 -> index_link_0
- joint little_joint_0: child Link33 -> little_link_0
- joint little_joint_1: child Link34 -> little_link_1; parent Link33 -> little_link_0
- joint middle_joint_0: child Link13 -> middle_link_0
- joint middle_joint_1: child Link14 -> middle_link_1; parent Link13 -> middle_link_0
- joint ring_joint_0: child Link23 -> ring_link_0
- joint ring_joint_1: child Link24 -> ring_link_1; parent Link23 -> ring_link_0
- joint thumb_joint_0: child Link43 -> thumb_link_0
- joint thumb_joint_1: child Link44 -> thumb_link_1; parent Link43 -> thumb_link_0
- joint thumb_joint_2: child Link47 -> thumb_link_2; parent Link44 -> thumb_link_1
- joint thumb_joint_3: child Link48 -> thumb_link_3; parent Link47 -> thumb_link_2

Commit message: modify the kuka_inspirehand task to solely depend on PD control without low-level fabric controller

File: dextrah_lab/assets/kuka_inspirehand/urdf/combined.urdf (robot description, URDF)
Before this commit: robot lbr_iiwa7_r800, 22 links, 21 joints
Links:
- added link index_tip, mass 1e-6
- added link little_tip, mass 1e-6
- added link middle_tip, mass 1e-6
- added link ring_tip, mass 1e-6
- added link thumb_tip, mass 1e-6
Joints:
- added joint index_tip_fixed: type fixed, parent index_link_1, child index_tip, origin xyz=0.005 0.035 0.002 rpy=0 0 0
- added joint little_tip_fixed: type fixed, parent little_link_1, child little_tip, origin xyz=0.005 0.035 0.003 rpy=0 0 0
- added joint middle_tip_fixed: type fixed, parent middle_link_1, child middle_tip, origin xyz=0.005 0.035 0.002 rpy=0 0 0
- added joint ring_tip_fixed: type fixed, parent ring_link_1, child ring_tip, origin xyz=0.005 0.035 0.002 rpy=0 0 0
- added joint thumb_tip_fixed: type fixed, parent thumb_link_3, child thumb_tip, origin xyz=-0.01 0.015 0.005 rpy=0 0 0
